File: board_tape_i2c.kicad_sch (KiCad schematic)
At the start: 25 parts, among them J1 C64-CassettePort, J10 Power for external devices, J2 Conn_01x04_Socket, J3 Conn_01x04_Socket, J4 Conn_01x04_Socket, J5 Conn_01x04_Socket, J6 Conn_01x04, J7 Conn_01x04, J8 Conn_01x04, J9 Conn_01x04, Q1 BSS138W, Q2 BSS138W, U1 XC6206P332MR

Commit message: Version 0.2
SDA and SCL reversed in cassette port

Signed-off-by: Timo Voutilainen <voutti@users.noreply.github.com>
Parts:
- removed JP2: SolderJumper_2_Open, Jumper:SolderJumper-2_P1.3mm_Open_RoundedPad1.0x1.5mm, symbol Jumper:SolderJumper_2_Open
- added H1, H2: MountingHole, TiVo_Library:MountingHole_3.2mm_M3_Reduced, symbol Mechanical:MountingHole
- added JP2: SolderJumper_2_Bridged, Jumper:SolderJumper-2_P1.3mm_Bridged2Bar_RoundedPad1.0x1.5mm, symbol Jumper:SolderJumper_2_Bridged
- F1, J1, J10, J2, J3, J4, J5, J6, J7, J8, J9: now not fitted; now left out of the parts list
- R1, R2, R3, R4: value 4k7 -> 10k
Connections:
- net SCL_5V: now also R8.2; no longer R7.2
- net SDA_5V: now also R7.2, JP2.1 (A); no longer R8.2
- net at R4.2: now also JP2.2 (B)
- no-connect marks 12 -> 4
Other:
- note added: "C64 Cassette port sense line has a strong 3.3kOhm pull-up so, normally you don't want any more pull-ups on 5V side. Therefore JP1 is open."
- title: (none) -> C64 Cassette port I2C adapter
- moved on the sheet: Q1, Q2, R1, R2, R3, R4
